Commit message: 10282231

File: src/urdf/irb1600.urdf (robot description, URDF)
Before this commit: robot abb_irb1600_6_12, 10 links, 9 joints
Links:
- removed link tool0
- added link PowerScan; collision mesh filename=package://view_planner/model/PowerScan_small.stl; visual mesh filename=package://view_planner/model/PowerScan_small.stl
Joints:
- removed joint link_6-tool0
- added joint link_6-PowerScan: type fixed, parent flange, child PowerScan, origin xyz=0 0 0 rpy=0 1.5707963267948966 0
